File: PCB/Nodo_sensor_nodemcu/Nodo_sensor_nodemcu.sch (KiCad schematic (older format))
At the start: 3 parts

Commit message: pcb
Parts:
- Conector_sensores1: renamed from Conector_sensores; value Conn_01x05 -> Conector_sensores; footprint (none) -> Connector_PinSocket_2.54mm:PinSocket_1x05_P2.54mm_Vertical; symbol Conn_01x05 -> Nodo_sensor_nodemcu-rescue:Conn_01x05
- Entrada_5V1: renamed from Entrada_5V; value Conn_01x02 -> Entrada_5V; footprint (none) -> TerminalBlock:TerminalBlock_bornier-2_P5.08mm; symbol Conn_01x02 -> Nodo_sensor_nodemcu-rescue:Conn_01x02
- NodeMCU_V2: footprint (none) -> nodemcu:NodeMCU_Amica_R2; symbol NodeMCU_Amica_R2 -> Nodo_sensor_nodemcu-rescue:NodeMCU_Amica_R2
Connections:
- wire segments 18 -> 14
Changed lines of the file:
@@
-EESchema Schematic File Version 2
-LIBS:power
-LIBS:device
-LIBS:switches
-LIBS:relays
-LIBS:motors
-LIBS:transistors
-LIBS:conn
-LIBS:linear
-LIBS:regul
-LIBS:74xx
-LIBS:cmos4000
-LIBS:adc-dac
-LIBS:memory
-LIBS:xilinx
-LIBS:microcontrollers
-LIBS:dsp
-LIBS:microchip
-LIBS:analog_switches
-LIBS:motorola
-LIBS:texas
-LIBS:intel
-LIBS:audio
-LIBS:interface
-LIBS:digital-audio
-LIBS:philips
-LIBS:display
-LIBS:cypress
-LIBS:siliconi
-LIBS:opto
-LIBS:atmel
-LIBS:contrib
-LIBS:valves
-LIBS:nodemcu
-EELAYER 25 0
+EESchema Schematic File Version 4
+LIBS:Nodo_sensor_nodemcu-cache
+EELAYER 29 0
 EELAYER END
 $Descr A4 11693 8268
@@
 $EndDescr
 $Comp
-L NodeMCU_Amica_R2 NodeMCU_V2
+L Nodo_sensor_nodemcu-rescue:NodeMCU_Amica_R2 NodeMCU_V2
 U 1 1 5CD081FB
 P 2600 3250
-F 0 "NodeMCU_V2" H 2600 4050 50  0000 C CNN
+F 0 "NodeMCU_V2" H 2600 4050 50  0001 C CNN
 F 1 "NodeMCU_Amica_R2" H 2600 2400 50  0000 C CNN
-F 2 "" H 2850 3250 50  0000 C CNN
+F 2 "nodemcu:NodeMCU_Amica_R2" H 2850 3250 50  0001 C CNN
 F 3 "" H 2850 3250 50  0000 C CNN
 	1    2600 3250
@@
 $EndComp
 $Comp
-L Conn_01x05 Conector_sensores
+L Nodo_sensor_nodemcu-rescue:Conn_01x05 Conector_sensores1
 U 1 1 5CD083E8
 P 4700 2700
-F 0 "Conector_sensores" H 4700 3000 50  0000 C CNN
-F 1 "Conn_01x05" H 4700 2400 50  0000 C CNN
-F 2 "" H 4700 2700 50  0001 C CNN
+F 0 "Conector_sensores1" H 4700 3000 50  0001 C CNN
+F 1 "Conector_sensores" H 4700 2400 50  0000 C CNN
+F 2 "Connector_PinSocket_2.54mm:PinSocket_1x05_P2.54mm_Vertical" H 4700 2700 50  0001 C CNN
 F 3 "" H 4700 2700 50  0001 C CNN
 	1    4700 2700
 	1    0    0    -1
 $EndComp
+Text Label 4050 2600 0    60   ~ 0
+3V3
 Text Label 4050 2500 0    60   ~ 0
-3V3
-Text Label 4050 2600 0    60   ~ 0
 GND
 Text Label 4050 2700 0    60   ~ 0
@@
 LDR
 Wire Wire Line
-	4050 2500 4500 2500
+	4050 2600 4500 2600
 Wire Wire Line
-	4500 2600 4050 2600
+	4500 2500 4050 2500
 Wire Wire Line
 	4500 2700 4050 2700
@@
 Wire Wire Line
 	4500 2900 4050 2900
-Wire Wire Line
-	2150 3550 1700 3550
-Wire Wire Line
-	2150 3450 1700 3450
 Wire Wire Line
 	2150 3950 1700 3950
@@
 Text Label 1700 2550 0    60   ~ 0
 LDR
-Text Label 1700 3450 0    60   ~ 0
-GND
-Text Label 1700 3550 0    60   ~ 0
-3V3
 Text Label 1700 3850 0    60   ~ 0
 GND
@@
 5V
 $Comp
-L Conn_01x02 Entrada_5V
+L Nodo_sensor_nodemcu-rescue:Conn_01x02 Entrada_5V1
 U 1 1 5CD08548
 P 4700 3400
-F 0 "Entrada_5V" H 4700 3500 50  0000 C CNN
-F 1 "Conn_01x02" H 4700 3200 50  0000 C CNN
-F 2 "" H 4700 3400 50  0001 C CNN
+F 0 "Entrada_5V1" H 4700 3500 50  0001 C CNN
+F 1 "Entrada_5V" H 4700 3200 50  0000 C CNN
+F 2 "TerminalBlock:TerminalBlock_bornier-2_P5.08mm" H 4700 3400 50  0001 C CNN
 F 3 "" H 4700 3400 50  0001 C CNN
 	1    4700 3400
@@
 Wire Wire Line
 	3050 3150 3500 3150
-Wire Wire Line
-	3050 3850 3500 3850
-Wire Wire Line
-	3050 3950 3500 3950
 Text Label 3350 3050 0    60   ~ 0
 3V3
 Text Label 3350 3150 0    60   ~ 0
 GND
-Text Label 3350 3850 0    60   ~ 0
-GND
-Text Label 3350 3950 0    60   ~ 0
-3V3
 $EndSCHEMATC
